File: Hardware/APDS-9960_RGB_and_Gesture_Sensor.sch (EAGLE design)
At the start: 19 parts, among them U1 APDS-9960

Commit message: Updated version number to v10 for reds
Other:
- note added: "v10"
- note removed: "v02"
Changed lines of the file:
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@@
 <sheet>
 <plain>
-<text x="238.76" y="7.62" size="2.54" layer="94">v02</text>
+<text x="238.76" y="7.62" size="2.54" layer="94">v10</text>
 <text x="172.72" y="12.7" size="2.54" layer="94" align="center-left">Shawn Hymel</text>
 <rectangle x1="69.342" y1="116.332" x2="72.898" y2="117.348" layer="94"/>
